File: Dcf77_Elrad.sch (KiCad schematic (older format))
At the start: 54 parts, among them IC1 RC4558, IC2 LM393, IC3 TDA1572, IC4 4060N, IC5 L78L08, J1 uC, J2 KH, J4 AntIN, J5 12V, J6 12V ANT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

Commit message: add Libs
Parts:
- IC3: symbol TDA:TDA1572 -> Dcf77_Elrad-rescue:TDA1572-TDA
- IC4: symbol 40xx:4060N -> Dcf77_Elrad-rescue:4060N-40xx
Changed lines of the file:
@@
 $EndDescr
 $Comp
-L 40xx:4060N IC4
+L Dcf77_Elrad-rescue:4060N-40xx IC4
 U 1 1 61AB98E7
 P 9300 2300
@@
 $EndComp
 $Comp
-L 40xx:4060N IC4
+L Dcf77_Elrad-rescue:4060N-40xx IC4
 U 2 1 61ABAF8D
 P 6200 6950
@@
 	1600 5050 1950 5050
 $Comp
-L TDA:TDA1572 IC3
+L Dcf77_Elrad-rescue:TDA1572-TDA IC3
 U 1 1 61AE53D5
 P 6500 2450
